Commit message: Commit for project

File: Support/Collsions_Objects/Collision1.urdf (robot description, URDF)
Before this commit: robot cube, 1 links, 0 joints
Links:
- link baseLink: geometry collision mesh filename=Uniblate_25cm.stl scale=0.001 0.001 0.001; visual mesh filename=Uniblate_25cm.stl scale=0.001 0.001 0.001

File: Support/Ur5e_Urdf/urdf/UR_SSR.urdf (robot description, URDF)
Before this commit: robot ur5e, 11 links, 10 joints
Links:
- added link measurement_tool, mass 0.0; collision mesh filename=../Fin_grip_vhacd2.obj scale=0.02 0.02 0.02; visual mesh filename=../Fin_grip_vhacd2.obj scale=0.02 0.02 0.02
- added link tcp
Joints:
- added joint measurement_tool_joint: type fixed, parent tool0, child measurement_tool, origin xyz=0 0 0 rpy=0 3.14 0
- added joint tcp_joint: type fixed, parent measurement_tool, child tcp, origin xyz=0 0 0 rpy=0 0 0
